Commit message: Update g1 urdf mesh names

File: g1/g1_29dof_rev_1_0.urdf (robot description, URDF)
Before this commit: robot g1_29dof_rev_1_0, 39 links, 38 joints
Links:
- link torso_link: geometry collision mesh filename=meshes/torso_link.STL; visual mesh filename=meshes/torso_link.STL
- link waist_roll_link: geometry visual mesh filename=meshes/waist_roll_link.STL
- link waist_yaw_link: geometry visual mesh filename=meshes/waist_yaw_link.STL
